Commit message: Add collision geometry to all links

File: urdf/puma560_robot.urdf.xacro (robot description, xacro)
@@ -35,4 +35,11 @@
       <material name="green"/>
     </visual>
+    <collision>
+      <geometry>
+        <xacro:puma560_link_geometry link_num="1"/>
+      </geometry>
+      <origin rpy="0 0 ${M_PI/2}"/>
+      <material name="green"/>
+    </collision>
   </link>
   <link name="link2">
@@ -44,4 +51,11 @@
       <material name="red"/>
     </visual>
+    <collision>
+      <geometry>
+        <xacro:puma560_link_geometry link_num="2"/>
+      </geometry>
+      <origin xyz="0 0 -0.1" rpy="0 0 0"/>
+      <material name="red"/>
+    </collision>
   </link>
   <joint name="j1" type="revolute">
@@ -60,4 +74,11 @@
       <material name="blue"/>
     </visual>
+    <collision>
+      <geometry>
+        <xacro:puma560_link_geometry link_num="3"/>
+      </geometry>
+      <origin xyz="0 0 ${0.0435+d_2}"/>
+      <material name="blue"/>
+    </collision>
   </link>
   <joint name="j2" type="revolute">
@@ -76,4 +97,11 @@
       <material name="green"/>
     </visual>
+    <collision>
+      <geometry>
+        <xacro:puma560_link_geometry link_num="4"/>
+      </geometry>
+      <origin xyz="0 0 0" rpy="0 0 0"/>
+      <material name="green"/>
+    </collision>
   </link>
   <joint name="j3" type="revolute">
@@ -92,4 +120,11 @@
       <material name="red"/>
     </visual>
+    <collision>
+      <geometry>
+        <xacro:puma560_link_geometry link_num="5"/>
+      </geometry>
+      <origin xyz="0 0 ${d_4-0.071}" rpy="0 0 ${M_PI/2}"/>
+      <material name="red"/>
+    </collision>
   </link>
   <joint name="j4" type="revolute">
@@ -108,4 +143,11 @@
       <material name="green"/>
     </visual>
+    <collision>
+      <geometry>
+        <xacro:puma560_link_geometry link_num="6"/>
+      </geometry>
+      <origin xyz="0 0 0" rpy="${M_PI} 0 ${M_PI/2}"/>
+      <material name="green"/>
+    </collision>
   </link>
   <joint name="j5" type="revolute">
@@ -124,4 +166,11 @@
       <material name="blue"/>
     </visual>
+    <collision>
+      <geometry>
+        <xacro:puma560_link_geometry link_num="7"/>
+      </geometry>
+      <origin xyz="0 0 -0.010" rpy="0 0 0"/>
+      <material name="blue"/>
+    </collision>
   </link>
   <joint name="j6" type="revolute">

Commit message: Add link for mobile base

File: urdf/puma560_robot.urdf.xacro (robot description, xacro)
@@ -27,4 +27,24 @@
   <xacro:property name="a_5" value="0"/>
   <xacro:property name="a_6" value="0"/>
+  <link name="mobile_base">
+    <visual>
+      <geometry>
+        <cylinder length="0.5" radius="0.3"/>
+      </geometry>
+      <origin xyz="0 0 -0.25" rpy="0 0 0"/>
+      <color rgba="0.8 0.8 0.8 0.8"/>
+    </visual>
+    <collision>
+      <geometry>
+        <cylinder length="0.6" radius="0.2"/>
+      </geometry>
+      <origin xyz="0 0 -0.25" rpy="0 0 0"/>
+      <color rgba="0.8 0.8 0.8 0.8"/>
+    </collision>
+  </link>
+  <joint name="base_to_link1" type="fixed">
+    <parent link="mobile_base"/>
+    <child link="link1"/>
+  </joint>
   <link name="link1">
     <visual>

Commit message: Update planar joint for base

File: urdf/puma560_robot.urdf.xacro (robot description, xacro)
@@ -27,4 +27,29 @@
   <xacro:property name="a_5" value="0"/>
   <xacro:property name="a_6" value="0"/>
+  <!-- Make a planar joint with the world by hand -->
+  <link name="world" />
+  <link name="planar_x_link" />
+  <link name="planar_y_link" />
+  <joint name="planar_x_joint" type="prismatic">
+    <parent link="world"/>
+    <child link="planar_x_link"/>
+    <origin xyz="0 0 0" rpy="0 0 0"/>
+    <axis xyz="1 0 0"/>
+    <limit effort="10" velocity="1" lower="-10" upper="10" />
+  </joint>
+  <joint name="planar_y_joint" type="prismatic">
+    <parent link="planar_x_link"/>
+    <child link="planar_y_link"/>
+    <origin xyz="0 0 0" rpy="0 0 0"/>
+    <axis xyz="0 1 0"/>
+    <limit effort="10" velocity="1" lower="-10" upper="10" />
+  </joint>
+  <joint name="planar_yaw_joint" type="revolute">
+    <parent link="planar_y_link"/>
+    <child link="mobile_base"/>
+    <origin xyz="0 0 0" rpy="0 0 0"/>
+    <axis xyz="0 0 1"/>
+    <limit effort="10" velocity="1" lower="${-2*3.1415}" upper="${2*3.1415}" />
+  </joint>
   <link name="mobile_base">
     <visual>
